Commit message: waypoint_manager, localization, launch, multilayer_planning runtime bugs fixing

File: src/urdf/urdf/av21_description/urdf/av21.urdf (robot description, URDF)
Before this commit: robot AV21, 18 links, 17 joints
Joints:
- joint camera_front_right_joint: parent rear_axle_middle_ground -> rear_axle_middle

Commit message: QOS as constants and standardized among the nodes. Joystick-simulator setup. CSL enabled to joystick override.

File: src/urdf/urdf/av21_description/urdf/av21.urdf (robot description, URDF)
Before this commit: robot AV21, 18 links, 17 joints
Links:
- added link base_link
Joints:
- added joint center_of_gravity_joint: type fixed, parent base_link, child center_of_gravity, origin xyz=0 0 0
